File: pcb/juksautin.kicad_pcb (KiCad board)
At the start: 2 copper layers, 65 x 35 mm, 20 parts, among them J1 Screw_Terminal_01x09, J2 ATMEGA32U4 pin 42, U1 SP3485CN, U2 LM4041, U3 R-78E5.0-0.5

Commit message: pcb: Random changes in Atmega32u4 board
Routing:
- net TX_EN: track 23.3 -> 17.6 mm, vias 0 -> 1
- net B: track 26.0 -> 24.6 mm
- net A: track 28.7 -> 27.9 mm, vias 0 -> 2
- net GND: vias 12 -> 13
